File: PCB/smarttle_v1.brd (EAGLE design)
At the start: 46.7 x 80 mm, 30 parts, among them IC1 THS4211, J1 USB-MICROB, U1 STM32F0_LQFP64, U2 SPX3819-3.3

Commit message: More updates
Parts:
- added C1, C3: 10nF, microbuilder:0805-NO
- added H1, H2, H3, H4: MOUNT-HOLE2.8, holes:2,8
- added R2, R3: (no value), resistor:R0603
- moved LED1 39.0 mm to (40.6, 19.1)
- moved R9 35.8 mm to (36.8, 19.1), turned to 180 degrees
- moved U1 20.7 mm to (12.7, 15.2)
- moved LCD 16.9 mm to (41.9, 50.8)
- moved KEYPAD 16.9 mm to (41.9, 31.8)
- moved PWM 8.98 mm to (8.89, 68.6)
- moved LED2 4.02 mm to (40.6, 15.2)
- moved JP1 2.54 mm to (16.5, 3.81)
- moved R8 2.54 mm to (36.8, 16.5), turned to 180 degrees
Connections:
- new net BOOT0: R2.2, U1.60
- net +3V3: now also C1.1, C3.1, R3.2, U1.13, U1.32, U1.64
- net GND: now also C1.2, C3.2, R2.1, U1.12, U1.31, U1.63
- net NRST: now also R3.1, U1.7
Routing:
- net +5V: track 17.5 -> 20.7 mm
Other:
- board size 46.7 x 80 mm -> 44.1 x 80 mm
