File: PCB/smarttle_v1.sch (EAGLE design)
At the start: 30 parts, among them IC1 THS4211, J1 USB-MICROB, U1 STM32F0_LQFP64, U2 SPX3819-3.3

Commit message: More updates
Parts:
- added C1, C3: 10nF, microbuilder:CAP_CERAMIC0805-NOOUTLINE
- added H1, H2, H3, H4: MOUNT-HOLE2.8, holes:MOUNT-HOLE2.8
- added R2, R3: (no value), resistor:R-US_R0603
Connections:
- new net BOOT0: R2.2, U1G$1.BOOT0
- net +3V3: now also C1.1, C3.1, R3.2, U1G$1.VDD, U1G$1.VDDA
- net GND: now also C1.2, C3.2, R2.1, U1G$1.VSS, U1G$1.VSSA
- net NRST: now also R3.1, U1G$1.NRST
Other:
- moved on the sheet: U1G$2, U1G$3, U1G$4, U1G$5
