File: PCB/boilup_v3.sch (EAGLE design)
At the start: 50 parts, among them U1 STM32F0_LQFP64, U2 SPX3819-3.3

Commit message: v3 using i2c and a level shifter
Parts:
- added U$5: TXS0102, smarttle:TXS0102
Connections:
- removed net MISO: U1G$2.PA6
- removed net MOSI: LCD.4, U1G$2.PA7
- removed net SCK: LCD.3, U1G$2.PA5
- new net I2C2_SCL: REDUNDANT.7, U$5.B1, U1G$5.PF6
- new net I2C2_SDA: REDUNDANT.5, U$5.A1, U1G$5.PF7
- new net SCL: LCD.3, U$5.B2
- new net SDA: LCD.4, U$5.A2
- net +3V3: now also U$5.OE, U$5.VCCA
- net +5V: now also U$5.VCCB
- net GND: now also U$5.GND
Other:
- moved on the sheet: REDUNDANT
Changed lines of the file:
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@@
 <part name="3V3" library="led" library_urn="urn:adsk.eagle:library:259" deviceset="LED" device="SML0805" package3d_urn="urn:adsk.eagle:package:15830/1"/>
 <part name="R5" library="resistor" library_urn="urn:adsk.eagle:library:348" deviceset="R-US_" device="R0603" package3d_urn="urn:adsk.eagle:package:26057/1"/>
+<part name="U$5" library="smarttle" deviceset="TXS0102" device=""/>
+<part name="+3V6" library="supply1" library_urn="urn:adsk.eagle:library:371" deviceset="+3V3" device=""/>
+<part name="P+6" library="supply1" library_urn="urn:adsk.eagle:library:371" deviceset="+5V" device=""/>
+<part name="+3V7" library="supply1" library_urn="urn:adsk.eagle:library:371" deviceset="+3V3" device=""/>
+<part name="GND8" library="supply1" library_urn="urn:adsk.eagle:library:371" deviceset="GND" device=""/>
 </parts>
 <sheets>
@@
 <instance part="C1" gate="G$1" x="55.88" y="93.98"/>
 <instance part="C3" gate="G$1" x="63.5" y="93.98"/>
-<instance part="REDUNDANT" gate="A" x="210.82" y="236.22"/>
+<instance part="REDUNDANT" gate="A" x="248.92" y="238.76"/>
 <instance part="BUTTON" gate="G$1" x="71.12" y="40.64"/>
 <instance part="R12" gate="G$1" x="71.12" y="48.26" rot="R90"/>
@@
 <instance part="3V3" gate="G$1" x="205.74" y="33.02"/>
 <instance part="R5" gate="G$1" x="205.74" y="43.18" rot="R90"/>
+<instance part="U$5" gate="G$1" x="208.28" y="238.76"/>
+<instance part="+3V6" gate="G$1" x="193.04" y="251.46"/>
+<instance part="P+6" gate="1" x="223.52" y="251.46"/>
+<instance part="+3V7" gate="G$1" x="193.04" y="233.68"/>
+<instance part="GND8" gate="1" x="220.98" y="226.06"/>
 </instances>
 <busses>
@@
 <segment>
 <pinref part="REDUNDANT" gate="A" pin="4"/>
-<wire x1="215.9" y1="238.76" x2="220.98" y2="238.76" width="0.1524" layer="91"/>
-<label x="220.98" y="238.76" size="1.778" layer="95"/>
+<wire x1="254" y1="241.3" x2="259.08" y2="241.3" width="0.1524" layer="91"/>
+<label x="259.08" y="241.3" size="1.778" layer="95"/>
 </segment>
 </net>
@@
 <segment>
 <pinref part="REDUNDANT" gate="A" pin="10"/>
-<wire x1="215.9" y1="231.14" x2="223.52" y2="231.14" width="0.1524" layer="91"/>
-<label x="220.98" y="231.14" size="1.778" layer="95"/>
+<wire x1="254" y1="233.68" x2="261.62" y2="233.68" width="0.1524" layer="91"/>
+<label x="259.08" y="233.68" size="1.778" layer="95"/>
 </segment>
 <segment>
@@
 <wire x1="165.1" y1="243.84" x2="172.72" y2="243.84" width="0.1524" layer="91"/>
 <label x="170.18" y="243.84" size="1.778" layer="95"/>
+</segment>
+<segment>
+<pinref part="U$5" gate="G$1" pin="GND"/>
+<wire x1="220.98" y1="231.14" x2="220.98" y2="228.6" width="0.1524" layer="91"/>
+<pinref part="GND8" gate="1" pin="GND"/>
 </segment>
 </net>
@@
 <wire x1="63.5" y1="99.06" x2="58.42" y2="99.06" width="0.1524" layer="91"/>
 <junction x="58.42" y="99.06"/>
+</segment>
+<segment>
+<pinref part="U$5" gate="G$1" pin="VCCA"/>
+<wire x1="195.58" y1="246.38" x2="193.04" y2="246.38" width="0.1524" layer="91"/>
+<wire x1="193.04" y1="246.38" x2="193.04" y2="248.92" width="0.1524" layer="91"/>
+<pinref part="+3V6" gate="G$1" pin="+3V3"/>
+</segment>
+<segment>
+<pinref part="U$5" gate="G$1" pin="OE"/>
+<wire x1="195.58" y1="231.14" x2="193.04" y2="231.14" width="0.1524" layer="91"/>
+<pinref part="+3V7" gate="G$1" pin="+3V3"/>
 </segment>
 </net>
@@
 <segment>
 <pinref part="REDUNDANT" gate="A" pin="1"/>
-<wire x1="208.28" y1="241.3" x2="200.66" y2="241.3" width="0.1524" layer="91"/>
-<label x="198.12" y="241.3" size="1.778" layer="95"/>
+<wire x1="246.38" y1="243.84" x2="238.76" y2="243.84" width="0.1524" layer="91"/>
+<label x="236.22" y="243.84" size="1.778" layer="95"/>
 </segment>
 <segment>
@@
 <wire x1="284.48" y1="104.14" x2="287.02" y2="104.14" width="0.1524" layer="91"/>
 </segment>
+<segment>
+<pinref part="U$5" gate="G$1" pin="VCCB"/>
+<wire x1="220.98" y1="246.38" x2="223.52" y2="246.38" width="0.1524" layer="91"/>
+<wire x1="223.52" y1="246.38" x2="223.52" y2="248.92" width="0.1524" layer="91"/>
+<pinref part="P+6" gate="1" pin="+5V"/>
+</segment>
 </net>
 <net name="ROW1" class="0">
@@
 <segment>
 <pinref part="REDUNDANT" gate="A" pin="8"/>
-<wire x1="215.9" y1="233.68" x2="223.52" y2="233.68" width="0.1524" layer="91"/>
-<label x="220.98" y="233.68" size="1.778" layer="95"/>
+<wire x1="254" y1="236.22" x2="261.62" y2="236.22" width="0.1524" layer="91"/>
+<label x="259.08" y="236.22" size="1.778" layer="95"/>
 </segment>
 <segment>
@@
 <segment>
 <pinref part="REDUNDANT" gate="A" pin="9"/>
-<wire x1="208.28" y1="231.14" x2="200.66" y2="231.14" width="0.1524" layer="91"/>
-<label x="193.04" y="231.14" size="1.778" layer="95"/>
+<wire x1="246.38" y1="233.68" x2="238.76" y2="233.68" width="0.1524" layer="91"/>
+<label x="231.14" y="233.68" size="1.778" layer="95"/>
 </segment>
 </net>
@@
 <segment>
 <pinref part="REDUNDANT" gate="A" pin="6"/>
-<wire x1="215.9" y1="236.22" x2="223.52" y2="236.22" width="0.1524" layer="91"/>
-<label x="220.98" y="236.22" size="1.778" layer="95"/>
+<wire x1="254" y1="238.76" x2="261.62" y2="238.76" width="0.1524" layer="91"/>
+<label x="259.08" y="238.76" size="1.778" layer="95"/>
 </segment>
 </net>
@@
 <segment>
 <pinref part="REDUNDANT" gate="A" pin="3"/>
-<wire x1="208.28" y1="238.76" x2="200.66" y2="238.76" width="0.1524" layer="91"/>
-<label x="198.12" y="238.76" size="1.778" layer="95"/>
-</segment>
-</net>
-<net name="SCK" class="0">
-<segment>
-<wire x1="53.34" y1="220.98" x2="50.8" y2="220.98" width="0.1524" layer="91"/>
-<label x="38.1" y="220.98" size="1.778" layer="95"/>
-<pinref part="U1" gate="G$2" pin="PA5"/>
-<wire x1="50.8" y1="220.98" x2="43.18" y2="220.98" width="0.1524" layer="91"/>
-<junction x="50.8" y="220.98"/>
-</segment>
-<segment>
-<pinref part="LCD" gate="A" pin="3"/>
-<wire x1="165.1" y1="238.76" x2="172.72" y2="238.76" width="0.1524" layer="91"/>
-<label x="170.18" y="238.76" size="1.778" layer="95"/>
-</segment>
-</net>
-<net name="MISO" class="0">
-<segment>
-<wire x1="53.34" y1="215.9" x2="50.8" y2="215.9" width="0.1524" layer="91"/>
-<label x="38.1" y="215.9" size="1.778" layer="95"/>
-<pinref part="U1" gate="G$2" pin="PA6"/>
-<wire x1="50.8" y1="215.9" x2="43.18" y2="215.9" width="0.1524" layer="91"/>
-<junction x="50.8" y="215.9"/>
-</segment>
-</net>
-<net name="MOSI" class="0">
-<segment>
-<wire x1="53.34" y1="210.82" x2="50.8" y2="210.82" width="0.1524" layer="91"/>
-<label x="38.1" y="210.82" size="1.778" layer="95"/>
-<pinref part="U1" gate="G$2" pin="PA7"/>
-<wire x1="50.8" y1="210.82" x2="43.18" y2="210.82" width="0.1524" layer="91"/>
-<junction x="50.8" y="210.82"/>
-</segment>
-<segment>
-<pinref part="LCD" gate="A" pin="4"/>
-<wire x1="165.1" y1="236.22" x2="172.72" y2="236.22" width="0.1524" layer="91"/>
-<label x="170.18" y="236.22" size="1.778" layer="95"/>
+<wire x1="246.38" y1="241.3" x2="238.76" y2="241.3" width="0.1524" layer="91"/>
+<label x="236.22" y="241.3" size="1.778" layer="95"/>
 </segment>
 </net>
@@
 <segment>
 <pinref part="REDUNDANT" gate="A" pin="2"/>
-<wire x1="215.9" y1="241.3" x2="220.98" y2="241.3" width="0.1524" layer="91"/>
-<label x="220.98" y="241.3" size="1.778" layer="95"/>
+<wire x1="254" y1="243.84" x2="259.08" y2="243.84" width="0.1524" layer="91"/>
+<label x="259.08" y="243.84" size="1.778" layer="95"/>
 </segment>
 </net>
@@
 </segment>
 </net>
+<net name="I2C2_SDA" class="0">
+<segment>
+<pinref part="U1" gate="G$5" pin="PF7"/>
+<wire x1="45.72" y1="132.08" x2="53.34" y2="132.08" width="0.1524" layer="91"/>
+<label x="48.26" y="132.08" size="1.778" layer="95"/>
+</segment>
+<segment>
+<pinref part="U$5" gate="G$1" pin="A1"/>
+<wire x1="195.58" y1="241.3" x2="190.5" y2="241.3" width="0.1524" layer="91"/>
+<label x="182.88" y="241.3" size="1.778" layer="95"/>
+</segment>
+<segment>
+<pinref part="REDUNDANT" gate="A" pin="5"/>
+<wire x1="246.38" y1="238.76" x2="238.76" y2="238.76" width="0.1524" layer="91"/>
+<label x="231.14" y="238.76" size="1.778" layer="95"/>
+</segment>
+</net>
+<net name="I2C2_SCL" class="0">
+<segment>
+<pinref part="U1" gate="G$5" pin="PF6"/>
+<wire x1="45.72" y1="137.16" x2="53.34" y2="137.16" width="0.1524" layer="91"/>
+<label x="48.26" y="137.16" size="1.778" layer="95"/>
+</segment>
+<segment>
+<pinref part="U$5" gate="G$1" pin="B1"/>
+<wire x1="195.58" y1="236.22" x2="190.5" y2="236.22" width="0.1524" layer="91"/>
+<label x="182.88" y="236.22" size="1.778" layer="95"/>
+</segment>
+<segment>
+<pinref part="REDUNDANT" gate="A" pin="7"/>
+<wire x1="246.38" y1="236.22" x2="238.76" y2="236.22" width="0.1524" layer="91"/>
+<label x="231.14" y="236.22" size="1.778" layer="95"/>
+</segment>
+</net>
+<net name="SCL" class="0">
+<segment>
+<pinref part="U$5" gate="G$1" pin="B2"/>
+<wire x1="220.98" y1="236.22" x2="226.06" y2="236.22" width="0.1524" layer="91"/>
+<label x="220.98" y="236.22" size="1.778" layer="95"/>
+</segment>
+<segment>
+<pinref part="LCD" gate="A" pin="3"/>
+<wire x1="165.1" y1="238.76" x2="172.72" y2="238.76" width="0.1524" layer="91"/>
+<label x="170.18" y="238.76" size="1.778" layer="95"/>
+</segment>
+</net>
+<net name="SDA" class="0">
+<segment>
+<pinref part="U$5" gate="G$1" pin="A2"/>
+<wire x1="220.98" y1="241.3" x2="226.06" y2="241.3" width="0.1524" layer="91"/>
+<label x="220.98" y="241.3" size="1.778" layer="95"/>
+</segment>
+<segment>
+<pinref part="LCD" gate="A" pin="4"/>
+<wire x1="165.1" y1="236.22" x2="172.72" y2="236.22" width="0.1524" layer="91"/>
+<label x="170.18" y="236.22" size="1.778" layer="95"/>
+</segment>
+</net>
